Commit message: Fix gripper slip with compliant pads and compare five motion planners

File: src/franka_description/robots/common/franka_hand_actuated.xacro (robot description, xacro)
@@ -1,6 +1,7 @@
 <?xml version="1.0" encoding="utf-8"?>
 <robot xmlns:xacro="http://www.ros.org/wiki/xacro" name="hand">
+  <xacro:include filename="$(find franka_description)/robots/common/compliant_finger_pad.xacro"/>
   <!-- safety_distance: Minimum safety distance in [m] by which the collision volumes are expanded and which is enforced during robot motions -->
-  <xacro:macro name="franka_hand_actuated" params="connected_to:='' arm_id:='panda' rpy:='0 0 0' xyz:='0 0 0' tcp_xyz:='0 0 0.1034' tcp_rpy:='0 0 0' safety_distance:=0 gazebo:=false description_pkg:=franka_description">
+  <xacro:macro name="franka_hand_actuated" params="connected_to:='' arm_id:='panda' rpy:='0 0 0' xyz:='0 0 0' tcp_xyz:='0 0 0.1034' tcp_rpy:='0 0 0' safety_distance:=0 gazebo:=false description_pkg:=franka_description compliant_pads:=false pad_stiffness:=10000 pad_damping:=1.4 pad_travel:=0.0015">
     <xacro:unless value="${connected_to == ''}">
       <joint name="${arm_id}_hand_joint" type="fixed">
@@ -50,4 +51,5 @@
         </geometry>
       </collision>
+      <xacro:unless value="${compliant_pads}">
       <!-- rubber tip with which to grasp -->
       <collision>
@@ -57,4 +59,9 @@
         </geometry>
       </collision>
+      </xacro:unless>
+      <xacro:if value="${compliant_pads}">
+        <!-- Recessed backing: tiles move into this envelope on compression. -->
+        <collision><origin xyz="0 0.00858 0.04525"/><geometry><box size="0.0175 0.0132 0.0185"/></geometry></collision>
+      </xacro:if>
       <xacro:if value="${gazebo}">
         <xacro:inertial_props name="leftfinger" />
@@ -89,4 +96,5 @@
         </geometry>
       </collision>
+      <xacro:unless value="${compliant_pads}">
       <!-- rubber tip with which to grasp -->
       <collision>
@@ -96,4 +104,9 @@
         </geometry>
       </collision>
+      </xacro:unless>
+      <xacro:if value="${compliant_pads}">
+        <!-- Recessed backing: tiles move into this envelope on compression. -->
+        <collision><origin xyz="0 -0.00858 0.04525"/><geometry><box size="0.0175 0.0132 0.0185"/></geometry></collision>
+      </xacro:if>
       <xacro:if value="${gazebo}">
         <xacro:inertial_props name="rightfinger" />
@@ -104,5 +117,5 @@
       <child link="${arm_id}_leftfinger" />
       <origin xyz="0 0 0.0584" rpy="0 0 0" />
-      <axis xyz="0 1 0"/><limit lower="0" upper="0.04" effort="5" velocity="0.1"/>
+      <axis xyz="0 1 0"/><limit lower="0" upper="0.04" effort="10" velocity="0.1"/>
       <dynamics damping="0.1" friction="0.0"/>
    </joint>
@@ -111,7 +124,11 @@
      <child link="${arm_id}_rightfinger" />
      <origin xyz="0 0 0.0584" rpy="0 0 0" />
-     <axis xyz="0 -1 0"/><limit lower="0" upper="0.04" effort="5" velocity="0.1"/>
+     <axis xyz="0 -1 0"/><limit lower="0" upper="0.04" effort="10" velocity="0.1"/>
      <dynamics damping="0.1" friction="0.0"/>
    </joint>
+    <xacro:if value="${compliant_pads}">
+      <xacro:compliant_finger_pad parent="${arm_id}_leftfinger" side="1" stiffness="${pad_stiffness}" damping="${pad_damping}" travel="${pad_travel}"/>
+      <xacro:compliant_finger_pad parent="${arm_id}_rightfinger" side="-1" stiffness="${pad_stiffness}" damping="${pad_damping}" travel="${pad_travel}"/>
+    </xacro:if>
     <gazebo reference="${arm_id}_leftfinger"><mu1>1.5</mu1><mu2>1.5</mu2></gazebo>
     <gazebo reference="${arm_id}_rightfinger"><mu1>1.5</mu1><mu2>1.5</mu2></gazebo>

File: src/franka_description/robots/panda/panda_sim.urdf.xacro (robot description, xacro)
@@ -1,4 +1,8 @@
 <?xml version="1.0"?>
 <robot xmlns:xacro="http://www.ros.org/wiki/xacro" name="panda">
+  <xacro:arg name="compliant_pads" default="false"/>
+  <xacro:arg name="pad_stiffness" default="10000"/>
+  <xacro:arg name="pad_damping" default="1.4"/>
+  <xacro:arg name="pad_travel" default="0.0015"/>
   <xacro:include
     filename="$(find franka_description)/robots/common/franka_arm.xacro"/>
@@ -14,4 +18,8 @@
     tcp_rpy="0 0 0"
     safety_distance="0"
+    compliant_pads="$(arg compliant_pads)"
+    pad_stiffness="$(arg pad_stiffness)"
+    pad_damping="$(arg pad_damping)"
+    pad_travel="$(arg pad_travel)"
     gazebo="true"/>
   <link name="world"/>

File: src/panda_planning/worlds/world.urdf (robot description, URDF)
Before this commit: robot panda_obstacle_world, 28 links, 27 joints
Links:
- link place_bin_back: geometry collision box size=0.304 0.035 0.1; visual box size=0.304 0.035 0.1
- link rack_lower: geometry collision box size=0.418 0.26 0.05; visual box size=0.418 0.26 0.05
- link rack_upper: geometry collision box size=0.418 0.26 0.05; visual box size=0.418 0.26 0.05
Joints:
- joint center_partition_fixed: origin xyz=0.46 -0.08 0.21 rpy=0 0 0 -> xyz=0.46 -0.12 0.21 rpy=0 0 0
- joint pillar_right_fixed: origin xyz=0.54 -0.32 0.275 rpy=0 0 0 -> xyz=0.60 -0.32 0.275 rpy=0 0 0
